File: Christmast Ornament.kicad_pcb (KiCad board)
At the start: 2 copper layers, 98.8 x 98.7 mm, 62 parts, among them J1 USB_OTG, J2 CONN_01X06, Q1 8205A, Q2 SI2302, Q3 BC817, SW1 SW_Push, SW2 SW_Push, U1 TP4056, U10 WS2812b, U2 HT7833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

Commit message: Silkscreen text changed
Other:
- board text added: "SSID: Arbolito"
- board text removed: "SSID: Arbolito Passw: qwerty"
Changed lines of the file:
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@@
     )
   )
-  (gr_text "SSID: Arbolito\nPassw: qwerty" (at 168.041 89.281) (layer B.SilkS)
+  (gr_text "SSID: Arbolito" (at 168.041 89.281) (layer B.SilkS)
     (effects (font (size 0.8 0.8) (thickness 0.15)) (justify mirror))
   )

Commit message: Added text for the custemer Id
Other:
- board text added: "JLCJLCJLCJLC"
Changed lines of the file:
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@@
     (area 118.662046 37.751949 217.545316 136.571691)
     (thickness 1.6)
-    (drawings 770)
+    (drawings 771)
     (tracks 544)
     (zones 0)
@@
     (aux_axis_origin 0 0)
     (grid_origin 167.406 129.921)
-    (visible_elements FFFFFF5F)
+    (visible_elements FFFFEF5F)
     (pcbplotparams
       (layerselection 0x010f0_80000001)
@@
     )
   )
+  (gr_text JLCJLCJLCJLC (at 164.993 116.84) (layer B.SilkS)
+    (effects (font (size 1.5 1.5) (thickness 0.3)) (justify mirror))
+  )
   (gr_text "SSID: Arbolito" (at 168.041 89.281) (layer B.SilkS)
